File: board/bleriot-simsens.kicad_sch (KiCad schematic)
At the start: 24 parts, among them J3 POWER, J4 RS485, U1 LM1117MP-3.3, U4 MAX485E, U5 PAN2110P0AA, U6 PY32F030F1xPx, X2 SWD, Y2 16MHz

Commit message: WIP
Parts:
- removed C7: 100n, Capacitor_SMD:C_0805_2012Metric, symbol Device:C
- removed R1: 1k5, Resistor_SMD:R_0805_2012Metric, symbol Device:R
- removed U4: MAX485E, Package_SO:SOIC-8_3.9x4.9mm_P1.27mm, symbol Interface_UART:MAX485E
- added AC1: 100n, Capacitor_SMD:C_0805_2012Metric, symbol Device:C
- added AR1: 10k 0.1%, Resistor_SMD:R_0805_2012Metric, symbol Device:R
- added AR2: 4.02k 0.1%, Resistor_SMD:R_0805_2012Metric, symbol Device:R
- added AR3: 6.49k 0.1%, Resistor_SMD:R_0805_2012Metric, symbol Device:R
- J2: renamed from J4; value RS485 -> INPUT
- renumbered A2 to A1, C3 to C1, C8 to C2, C6 to C3, C9 to C4, C11 to C5, C10 to C6, C12 to C7, D3 to D2, D4 to D3, J3 to J1, R3 to R1, R4 to R2, U5 to U2, U6 to U3, X2 to X1, Y2 to Y1
Connections:
- net RS485_A is gone; now on net +5V: J2.3 (Pin_3)
- net +3V3: now also AR1.2
- net GND: now also AC1.2, AR3.1
- net RF_DATA: now also U3.17 (PB5); no longer U3.6 (PA3)
- net RF_SCK: now also U3.11 (PA9-OSC32OUT); no longer U3.5 (PA2)
- net ~{RF_CS}: now also U3.12 (PA10-OSC32IN); no longer U3.4 (PF3)
- net RS485_B renamed INPUT_RAW
- net INPUT_RAW: now also AR1.1, AR2.2
- net RS485_RX: no longer names the net of U3.19 (PB7)
- net RS485_RX: no longer D1.3 (COM)
- net RS485_TX: no longer names the net of U3.18 (PB6)
- net RS485_TXEN: no longer names the net of U3.20 (PF4-BOOT0)
- new net INPUT_MCU: AC1.1, AR2.1, AR3.2, D1.3 (COM), U3.5 (PA2)
- no-connect marks 9 -> 11
Other:
- moved on the sheet: D1
