File: board/bleriot-sense.kicad_sch (KiCad schematic)
At the start: 24 parts, among them J1 POWER, J2 INPUT, U1 XC6206P332MR, U2 PAN2110P0AA, U3 PY32F030F1xPx, X1 SWD, Y1 16MHz

Commit message: WIP
Parts:
- U2: footprint Package_TO_SOT_SMD:SOT-23-8 -> Drake:PAN211x_SOT23-8_P0.8mm
Changed lines of the file:
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@@
 			)
 		)
-		(property "Footprint" "Package_TO_SOT_SMD:SOT-23-8"
+		(property "Footprint" "Drake:PAN211x_SOT23-8_P0.8mm"
 			(at 97.79 72.898 0)
 			(hide yes)
