File: board/bleriot-sense.kicad_pcb (KiCad board)
At the start: 2 copper layers, 25 parts, among them J1 POWER, J2 INPUT, U1 LM1117MP-3.3, U2 PAN2110P0AA, U3 PY32F030F1xPx, X1 SWD, Y1 16MHz

Commit message: WIP
Parts:
- removed H1: MountingHole, MountingHole:MountingHole_3.7mm_Pad_Via
- C1, C3: value 10u -> 1u
- U1: value LM1117MP-3.3 -> XC6206P332MR; footprint Package_TO_SOT_SMD:SOT-223-3_TabPin2 -> Package_TO_SOT_SMD:SOT-23-3
- moved U1 0.48 mm to (101.6, 54.7)

Commit message: WIP
Parts:
- AC1: moved to B.Cu
- AR1: value 10k 0.1% -> 10k; moved to B.Cu
- AR2: value 4.02k 0.1% -> 4.02k; moved to B.Cu
- AR3: value 6.49k 0.1% -> 6.49k; moved to B.Cu
- U2: footprint Package_SO:SOIC-8_3.9x4.9mm_P1.27mm -> Package_TO_SOT_SMD:SOT-23-8
- moved J2 127.0 mm to (195.7, 106.0), turned to 90 degrees
- moved AC1 116.7 mm to (190.0, 105.0)
- moved AR3 105.0 mm to (190.0, 101.5), turned to 180 degrees
- moved AR2 104.8 mm to (190.0, 98.0)
- moved AR1 104.6 mm to (190.0, 94.5), turned to 180 degrees
- moved R2 102.7 mm to (188.5, 105.0)
- moved C5 98.0 mm to (182.0, 94.0), turned to 90 degrees
- moved A1 96.6 mm to (174.1, 106.4), turned to 180 degrees
- moved D3 93.3 mm to (188.5, 101.0), turned to 180 degrees
- moved R1 92.7 mm to (177.0, 103.0), turned to -90 degrees
- moved C2 92.2 mm to (169.0, 98.5), turned to 180 degrees
- moved C1 92.2 mm to (163.5, 103.5)
- moved C4 90.2 mm to (169.0, 100.5), turned to 180 degrees
- moved X1 89.0 mm to (182.5, 101.0), turned to 90 degrees
- moved D2 87.9 mm to (188.5, 101.0), turned to 180 degrees
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Routing:
- net +3V3: track 0.00 -> 70.3 mm, vias 0 -> 3
- net +5V: track 0.00 -> 65.4 mm
- net /INPUT_MCU: track 0.00 -> 30.6 mm, vias 0 -> 2
- net GND: track 0.00 -> 27.9 mm, vias 0 -> 63
- net /LED: track 0.00 -> 16.6 mm, vias 0 -> 2
- net /INPUT_RAW: track 0.00 -> 12.6 mm
- net /RF_DATA: track 0.00 -> 10.7 mm
- net Net-(U3-PA11): track 0.00 -> 10.2 mm, vias 0 -> 2
- net Net-(U3-PA13): track 0.00 -> 9.49 mm
- net /~{RF_CS}: track 0.00 -> 5.90 mm
- net Net-(U2-XC1): track 0.00 -> 5.33 mm
- net Net-(U3-PF2-NRST): track 0.00 -> 4.89 mm
- net Net-(U2-XC0): track 0.00 -> 4.34 mm
- net Net-(D3-K): track 0.00 -> 4.05 mm
- net /RF_SCK: track 0.00 -> 3.11 mm
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- added copper zone on B.Cu, net GND
- added copper zone on F.Cu, net GND
Other:
- board outline added: 63 x 22 mm
- board text added: "+5V"
- board text added: "Flow OC"
- board text added: "Flow PP"
- board text added: "GND"
- board text added: "IN"
- board text added: "NTC 10k B3950"
- board text added: "Press 0.5–5V"
- board text added: "bleriot-sense v1.0 drake.cz"
- board text added: "resistor tolerances: 0.1%"

Commit message: WIP
Parts:
- AR1: value 10k -> 10k 0.1%
- AR2: value 4.02k -> 4.02k 0.1%
- AR3: value 6.49k -> 6.49k 0.1%
- U2: footprint Package_TO_SOT_SMD:SOT-23-8 -> Drake:PAN211x_SOT23-8_P0.8mm
- moved A1 0.15 mm to (174.2, 106.4)
Routing:
- net GND: track 27.9 -> 31.4 mm, vias 63 -> 68
Other:
- board text added: "bleriot-sense v1.1 drake.cz"
- board text removed: "bleriot-sense v1.0 drake.cz"
