File: board/bleriot-sense.kicad_pcb (KiCad board)
At the start: 2 copper layers, 63 x 22 mm, 19 parts, among them J1 POWER, J2 INPUT, U1 XC6206P332MR, U2 PAN2110P0AA, U4 PY32F003L1xSx, X1 SWD, Y1 16MHz

Commit message: board fixes
Parts:
- J1: footprint Connector_Phoenix_MSTB:PhoenixContact_MSTBA_2,5_2-G_1x02_P5.00mm_Horizontal -> Connector_Phoenix_MC:PhoenixContact_MC_1,5_2-G-3.5_1x02_P3.50mm_Horizontal
- J2: footprint Connector_Phoenix_MSTB:PhoenixContact_MSTBA_2,5_3-G_1x03_P5.00mm_Horizontal -> Connector_Phoenix_MC:PhoenixContact_MC_1,5_3-G-3.5_1x03_P3.50mm_Horizontal
- moved C1 9.61 mm to (165.5, 94.0), turned to -90 degrees
- moved C3 9.57 mm to (173.5, 94.0), turned to -90 degrees
- moved X1 9.55 mm to (180.5, 94.0)
- moved U1 7.74 mm to (169.5, 94.0), turned to 180 degrees
- moved J1 6.21 mm to (164.4, 99.3)
- moved J2 1.56 mm to (195.6, 104.4)
Routing:
- net +5V: track 65.9 -> 55.4 mm
- net Net-(U4-PB5/PA14-SWC): track 28.9 -> 19.0 mm
- net Net-(U4-PA10/PA13-SWD): track 26.3 -> 16.4 mm
- net +3V3: track 47.6 -> 39.4 mm
- net GND: track 17.8 -> 21.4 mm, vias 50 -> 55
Other:
- board size 63 x 22 mm -> 53 x 22 mm
- board text added: "bleriot-sense v1.1 drake.cz"
- board text removed: "bleriot-sense v1.0 drake.cz"
