File: board/bleriot-sense.kicad_pcb (KiCad board)
At the start: 2 copper layers, 53 x 22 mm, 19 parts, among them J1 POWER, J2 INPUT, U1 XC6206P332MR, U2 PAN2110P0AA, U4 PY32F003L1xSx, X1 SWD, Y1 16MHz

Commit message: Update design rules and component footprints in Bleriot Sense board
- Modified DRC exclusions for silk over copper layers to adjust coordinates.
- Added a new DRC exclusion for starved thermal connections.
- Changed the footprint of the RF antenna from right to left orientation.
- Updated connector footprints for Phoenix connectors to reflect correct part numbers and dimensions.
Parts:
- A1: footprint RF_Antenna:Texas_SWRA117D_2.4GHz_Right -> RF_Antenna:Texas_SWRA117D_2.4GHz_Left
- J1: footprint Connector_Phoenix_MC:PhoenixContact_MC_1,5_2-G-3.5_1x02_P3.50mm_Horizontal -> Connector_Phoenix_MSTB:PhoenixContact_MSTBA_2,5_2-G_1x02_P5.00mm_Horizontal
- J2: footprint Connector_Phoenix_MC:PhoenixContact_MC_1,5_3-G-3.5_1x03_P3.50mm_Horizontal -> Connector_Phoenix_MSTB:PhoenixContact_MSTBA_2,5_3-G_1x03_P5.00mm_Horizontal
- moved J2 1.59 mm to (195.2, 106.0)
- moved C1 1.12 mm to (166.0, 93.0), turned to 180 degrees
- moved J1 0.88 mm to (164.8, 98.5)
- moved U1 0.50 mm to (170.0, 94.0)
Routing:
- net +5V: track 55.4 -> 52.8 mm
- net +3V3: track 39.4 -> 38.9 mm
- net GND: track 21.4 -> 21.6 mm, vias 55 -> 59
Other:
- board size 53 x 22 mm -> 55 x 22 mm
- board text added: "bleriot-sense v1.2 drake.cz"
- board text removed: "bleriot-sense v1.1 drake.cz"
