File: board-ssop/bleriot-sense.kicad_sch (KiCad schematic)
At the start: 24 parts, among them J1 POWER, J2 INPUT, U1 XC6206P332MR, U2 PAN2110P0AA, U3 PY32F030F1xPx, X1 SWD, Y1 16MHz

Commit message: WIP
Parts:
- removed C5: 100n, Capacitor_SMD:C_0805_2012Metric, symbol Device:C
- removed D2: WS2812B, LED_SMD:LED_WS2812B_PLCC4_5.0x5.0mm_P3.2mm, symbol LED:WS2812B
- removed D3: LED, LED_SMD:LED_0805_2012Metric_Pad1.15x1.40mm_HandSolder, symbol Device:LED
- removed R1: 10k, Resistor_SMD:R_0805_2012Metric, symbol Device:R
- removed R2: 330R, Resistor_SMD:R_0805_2012Metric, symbol Device:R
- removed U3: PY32F030F1xPx, Package_SO:TSSOP-20_4.4x6.5mm_P0.65mm, symbol MCU_Puya_PY32F:PY32F030F1xPx
- added U4: PY32F003L1xSx, Package_SO:SOIC-8_3.9x4.9mm_P1.27mm, symbol MCU_Puya_PY32F:PY32F003L1xSx
- U2: footprint Package_TO_SOT_SMD:SOT-23-8 -> Package_SO:SOIC-8_3.9x4.9mm_P1.27mm; symbol Drake:PAN2110Z0AA -> Drake:PAN2110P0AA
Connections:
- net +3V3: now also U4.1 (VCC)
- net GND: now also U4.8 (VSS)
- net INPUT_MCU: now also U4.2 (PA0)
- net RF_DATA: now also U4.4 (PA2)
- net RF_SCK: now also U4.3 (PA1)
- net ~{RF_CS}: now also U4.5 (PB0/PF2-NRST)
- net at X1.1 (SWDIO): now also U4.6 (PA10/PA13-SWD)
- net at X1.3 (SWCLK): now also U4.7 (PB5/PA14-SWC)
- no-connect marks 11 -> 0
Other:
- moved on the sheet: C6, C7, X1
